File: Hardware/OpenMowerMainboard/OpenMowerMainboard.kicad_pcb (KiCad board)
At the start: 2 copper layers, 180 x 170 mm, 178 parts, among them IC1 74ALVC164245DGG,11, IC2 TSC101CILT, IC3 MAX20405AFOF_VY+T, J1 Conn_02x11_Top_Bottom, J10 Conn_01x05, J11 Conn_01x03_Male, J12 Conn_01x03_Male, J13 Conn_01x03_Male, J14 Conn_01x03_Male, J16 Conn_01x08, J17 Conn_01x02, J18 Conn_01x02, J19 Conn_01x04, J2 Conn_02x04_Top_Bottom, J20 Conn_01x10_Female, J21 Raspberry_Pi_2_3, J22 Conn_02x04_Odd_Even, J23 Conn_01x08, J3 Conn_01x02, J4 Conn_01x05, J5 Conn_01x04, J6 Conn_01x04, J7 Conn_01x04, J8 Conn_01x04, J9 Conn_01x04, M1 Fan, Q13 BSS138, Q14 BSS138, Q15 BSS138, Q16 BSS138, Q3 BSS138, Q5 BSS138, Q6 Q_PMOS_GDS, SW1 MK-11C04-G013, SW2 DA-01BP, U1 DNP, U10 74HC4051, U11 Pico, U2 MCP604, U3 SIP32509DT, U4 xESC2, U5 xESC2, U6 xESC2, U7 SN74LV1T34DBV, U9 74HC4051

Commit message: remove and test again
Parts:
- removed AC1201: LSM6DSOTR, MyModules:LGA-14_2.5X3X0.86_
- removed C1, C25, C5: 100nF, Capacitor_SMD:C_0805_2012Metric_Pad1.18x1.45mm_HandSolder
- removed C10: DNP, Capacitor_SMD:CP_Elec_10x12.5
- removed C11, C12: 4.7uF, Capacitor_SMD:C_1206_3216Metric
- removed C13, C14: 1uF, Capacitor_SMD:C_0805_2012Metric
- removed C15, C18, C19, C24, C26: 0.1uF, Capacitor_SMD:C_0603_1608Metric
- removed C16, C20, C21, C22: 22uF, Capacitor_SMD:C_1206_3216Metric
- removed C17: 2.2uF, Capacitor_SMD:C_0603_1608Metric
- removed C2, C3, C6, C7, C8: 220uF, Capacitor_THT:CP_Radial_D10.0mm_P5.00mm
- removed C23, C9: 680uF, Capacitor_SMD:CP_Elec_10x12.5
- removed D1: D_Schottky, Diode_SMD:D_SOD-123F
- removed D10, D11, D12, D4, D5, D6, D7, D8, D9: DNP, Diode_SMD:D_SMB
- removed D13, D14: DNP, Diode_SMD:D_SOD-123F
- removed D15, D16, D2, D3: D_Schottky, Diode_SMD:D_SMA_Handsoldering
- removed D17: DNP, Diode_SMD:D_0402_1005Metric_Pad0.77x0.64mm_HandSolder
- removed D18, D19, D20: DNP, Diode_SMD:D_SMA
- removed D23: LED, LED_SMD:LED_0805_2012Metric
- removed D25: WS2812B, LED_SMD:LED_WS2812B_PLCC4_5.0x5.0mm_P3.2mm
- removed F1: nSMD035-16V, lcsc:F1206
- removed F2, F4: Fuse, MyModules:Fuseholder5x20_horiz_open_inline_Type-I
- removed FID1, FID10, FID11, FID12, FID13, FID14, FID15, FID16, FID2, FID3, FID4, FID5, FID6, FID7, FID8, FID9: Fiducial, Fiducial:Fiducial_1mm_Mask2mm
- removed H1, H2, H3, H4: MountingHole_Pad, MountingHole:MountingHole_5mm_Pad_Via
- removed IC1: 74ALVC164245DGG,11, 74ALVC164245DGG:SOP50P810X120-48N
- removed IC2: TSC101CILT, TSC101CILT:SOT95P280X145-5N
- removed IC3: MAX20405AFOF_VY+T, MAX2040:MAX2040
- removed J1: Conn_02x11_Top_Bottom, Connector_Molex:Molex_Mini-Fit_Jr_5566-22A_2x11_P4.20mm_Vertical
- removed J10: Conn_01x05, Connector_JST:JST_PH_B5B-PH-K_1x05_P2.00mm_Vertical
- removed J11, J12, J13, J14: Conn_01x03_Male, Connector_JST:JST_XH_B3B-XH-A_1x03_P2.50mm_Vertical
- removed J16, J23: Conn_01x08, Connector_PinSocket_2.54mm:PinSocket_1x08_P2.54mm_Vertical
- removed J17, J18: Conn_01x02, Connector_JST:JST_XH_B2B-XH-A_1x02_P2.50mm_Vertical
- removed J19, J5, J6, J7, J8, J9: Conn_01x04, Connector_JST:JST_XH_B4B-XH-A_1x04_P2.50mm_Vertical
- removed J2: Conn_02x04_Top_Bottom, Connector_Molex:Molex_Mini-Fit_Jr_5566-08A_2x04_P4.20mm_Vertical
- removed J20: Conn_01x10_Female, Connector_PinHeader_2.54mm:PinHeader_1x10_P2.54mm_Vertical
- removed J21: Raspberry_Pi_2_3, lcsc:HDR-SMD_40P-P2.54-V-F-R2-C20-S8.8-EH
- removed J22: Conn_02x04_Odd_Even, Connector_PinHeader_2.54mm:PinHeader_2x04_P2.54mm_Vertical
- removed J3: Conn_01x02, Connector_Molex:Molex_Mini-Fit_Jr_5566-02A_2x01_P4.20mm_Vertical
- removed J4: Conn_01x05, Connector_JST:JST_XH_B5B-XH-A_1x05_P2.50mm_Vertical
- removed JP1, JP2, JP3, JP4, JP5: SolderJumper_3_Bridged12, Jumper:SolderJumper-3_P1.3mm_Bridged12_Pad1.0x1.5mm
- removed JP10, JP11: I2C_OR_TTL, Jumper:SolderJumper-3_P1.3mm_Bridged12_Pad1.0x1.5mm
- removed JP6, JP7, JP8: SolderJumper_2_Bridged, Jumper:SolderJumper-2_P1.3mm_Bridged_RoundedPad1.0x1.5mm
- removed JP9: SolderJumper_2_Open, Jumper:SolderJumper-2_P1.3mm_Open_RoundedPad1.0x1.5mm
- removed L1: 4.7uH 5A, Inductor_SMD:L_Vishay_IHLP-2525
- removed LOGO1: LOGO, Symbol:ESD-Logo_6.6x6mm_SilkScreen
- removed LOGO2: ESD-Logo_6.6x6mm_SilkScreen, Symbol:ESD-Logo_6.6x6mm_SilkScreen
- removed M1: Fan, Connector_PinHeader_2.54mm:PinHeader_1x02_P2.54mm_Vertical
- removed MH1, MH2, MH3, MH4, MH5, MH6, MH7, MH8: , MountingHole:MountingHole_2.7mm_M2.5
- removed Q13, Q14, Q15, Q16, Q3, Q5: BSS138, Package_TO_SOT_SMD:SOT-23
- removed Q6: Q_PMOS_GDS, Package_TO_SOT_SMD:TO-252-2
- removed R1, R12, R2, R26, R28, R4, R40, R42, R48, R50: 10k, Resistor_SMD:R_0805_2012Metric_Pad1.20x1.40mm_HandSolder
- removed R10, R13, R15, R16, R18, R19, R20, R3, R41, R43, R45, R47, R6, R7, R9: 1k, Resistor_SMD:R_0805_2012Metric_Pad1.20x1.40mm_HandSolder
- removed R11: 53k6 1%, Resistor_SMD:R_0805_2012Metric_Pad1.20x1.40mm_HandSolder
- removed R14, R17, R49: 4k7, Resistor_SMD:R_0805_2012Metric_Pad1.20x1.40mm_HandSolder
- removed R27, R5: 150, Resistor_SMD:R_0805_2012Metric_Pad1.20x1.40mm_HandSolder
- removed R44, R46: 47k, Resistor_SMD:R_0805_2012Metric_Pad1.20x1.40mm_HandSolder
- removed R51: 0.003R, Resistor_SMD:R_2512_6332Metric_Pad1.40x3.35mm_HandSolder
- removed R8: DNP, Resistor_SMD:R_0805_2012Metric_Pad1.20x1.40mm_HandSolder
- removed SW1: MK-11C04-G013, lcsc:SW-SMD_MK-11C04-G013
- removed SW2: DA-01BP, lcsc:SW-TH_DA-01BP
- removed TP1, TP2, TP5: TestPoint, TestPoint:TestPoint_Pad_D2.0mm
- removed U1: DNP, MyModules:LM2596S_MODULE
- removed U10, U9: 74HC4051, Package_SO:SSOP-16_4.4x5.2mm_P0.65mm
- removed U11: Pico, PicoW:Raspberry_Pi_Pico_SMT_THT
- removed U2: MCP604, Package_SO:SOIC-14_3.9x8.7mm_P1.27mm
- removed U3: SIP32509DT, Package_TO_SOT_SMD:SOT-23-6_Handsoldering
- removed U4, U5, U6: xESC2, xESC2:xESC2
- removed U7: SN74LV1T34DBV, Package_TO_SOT_SMD:SOT-23-5
- removed WT901: Conn_02x06_Female, MyModules:WT901
- removed XA1: Arduino_Uno_Shield, MyModules:Arduino_Uno_Shield
Routing:
- net +5V: track 887.6 -> 0.00 mm, vias 18 -> 0
- net +3V3: track 529.4 -> 0.00 mm, vias 18 -> 0
- net V_BATT: track 442.7 -> 0.00 mm, vias 31 -> 0
- net /IMU/MISO: track 216.3 -> 0.00 mm, vias 4 -> 0
- net /IMU/SCK: track 205.5 -> 0.00 mm, vias 2 -> 0
- net /IMU/MOSI: track 202.0 -> 0.00 mm, vias 2 -> 0
- net /RobotConnectors/SPEAKER_PLUS: track 197.8 -> 0.00 mm, vias 2 -> 0
- net /RobotConnectors/SPEAKER_MINUS: track 192.7 -> 0.00 mm, vias 2 -> 0
- net /IMU/~{CS}: track 186.9 -> 0.00 mm, vias 3 -> 0
- net /ESCs/ML_RX: track 168.6 -> 0.00 mm, vias 1 -> 0
- net /RaspberryPi/PICO_SWCLK: track 168.4 -> 0.00 mm, vias 1 -> 0
- net /RaspberryPi/PICO_SWDIO: track 161.5 -> 0.00 mm, vias 1 -> 0
- net /ESCs/ML_TX: track 158.7 -> 0.00 mm, vias 1 -> 0
- net Net-(U11-GPIO10): track 153.9 -> 0.00 mm, vias 6 -> 0
- net /ESCs/MC_RX: track 151.5 -> 0.00 mm, vias 1 -> 0
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- removed copper zone on B.Cu, net +5V
- removed copper zone on F.Cu, net +5V
- removed copper zone on B.Cu, net /ESCs/MC_PHASE_U
- removed copper zone on F.Cu, net /ESCs/MC_PHASE_U
- removed copper zone on B.Cu, net /ESCs/MC_PHASE_V
- removed copper zone on F.Cu, net /ESCs/MC_PHASE_V
- removed copper zone on B.Cu, net /ESCs/MC_PHASE_W
- removed copper zone on F.Cu, net /ESCs/MC_PHASE_W
- removed copper zone on B.Cu, net /ESCs/ML_PHASE_U
- removed copper zone on F.Cu, net /ESCs/ML_PHASE_U
- removed copper zone on B.Cu, net /ESCs/ML_PHASE_V
- removed copper zone on F.Cu, net /ESCs/ML_PHASE_V
- removed copper zone on B.Cu, net /ESCs/ML_PHASE_W
- removed copper zone on F.Cu, net /ESCs/ML_PHASE_W
- removed copper zone on B.Cu, net /ESCs/MR_PHASE_U
- removed copper zone on F.Cu, net /ESCs/MR_PHASE_U
- removed copper zone on B.Cu, net /ESCs/MR_PHASE_V
- removed copper zone on F.Cu, net /ESCs/MR_PHASE_V
- removed copper zone on B.Cu, net /ESCs/MR_PHASE_W
- removed copper zone on F.Cu, net /ESCs/MR_PHASE_W
- removed copper zone on F.Cu, net /RaspberryPi/RASPI_POWER
- removed copper zone on F.Cu, net /RobotConnectors/V_BATTERY
- removed copper zone on B.Cu, net GND
- removed copper zone on F.Cu, net GND
- removed copper zone on F.Cu, net Net-(IC3-LX_1)
- removed copper zone on B.Cu, net V_BATT
- removed copper zone on F.Cu, net V_BATT
Other:
- board outline removed
- board text removed: "3.3V"
- board text removed: "5V"
- board text removed: "5V,SIG,GND"
- board text removed: "5V,TRIG,ECHO,GND"
- board text removed: "Busy"
- board text removed: "Charge"
- board text removed: "GND"
- board text removed: "Hall 1"
- board text removed: "Hall 2"
- board text removed: "Hall 3"
- board text removed: "Hall 4"
- board text removed: "IOREF"
- board text removed: "Motor Connection"
- board text removed: "Mower Hall Sensors"
- board text removed: "OpenMower Mainboard ${git_version} License CC BY-NC-SA 4.0 https://github.com/ClemensElflein/OpenMower"
- board text removed: "Power Connection"
- board text removed: "RPi force power"
- board text removed: "RX"
- board text removed: "RXD"
- board text removed: "Rain"
- board text removed: "Speaker"
- board text removed: "Speaker +"
- board text removed: "Speaker -"
- board text removed: "TX"
- board text removed: "TXD"
- board text removed: "UI Board"
- board text removed: "USS 1"
- board text removed: "USS 2"
- board text removed: "USS 3"
- board text removed: "USS 4"
- board text removed: "USS 5"
- board text removed: "xESC Center"
- board text removed: "xESC Left"
- board text removed: "xESC Right"
