File: Hardware/OpenMowerMainboard/OpenMowerMainboard.kicad_sch (KiCad schematic)
At the start: 26 parts

Commit message: remove and test again
Parts:
- removed D23: LED, LED_SMD:LED_0805_2012Metric, symbol Device:LED
- removed FID1, FID10, FID11, FID12, FID13, FID14, FID15, FID16, FID2, FID3, FID4, FID5, FID6, FID7, FID8, FID9: Fiducial, Fiducial:Fiducial_1mm_Mask2mm, symbol Mechanical:Fiducial
- removed H1, H2, H3, H4: MountingHole_Pad, MountingHole:MountingHole_5mm_Pad_Via, symbol Mechanical:MountingHole_Pad
- removed R18, R41, R43: 1k, Resistor_SMD:R_0805_2012Metric_Pad1.20x1.40mm_HandSolder, symbol Device:R
- removed R40, R42: 10k, Resistor_SMD:R_0805_2012Metric_Pad1.20x1.40mm_HandSolder, symbol Device:R
Other:
- removed sheet ESCs
- removed sheet GPS
- removed sheet IMU
- removed sheet RaspberryPi
- removed sheet RobotConnectors
- removed sheet dcdc
- removed sheet opamps
- removed sheet pico
- removed sheet sound
- note removed: "Motor Connectors"
- note removed: "Sensor Connectors"
